File: eagle/TurnoutController/TurnoutController.brd (EAGLE design)
At the start: 61 x 48.3 mm, 19 parts, among them IC1 L293D, J1 POWER_JACKPTH

Commit message: 1.  Cleanup continues.  BlockController and the corresponding controller are deprecated along with SignalController and it's controller board.  These are replaced by the InputModule and OutputModule respectively 2.  TurnoutHandler moved to the MultiModuleController project folder 3.  Module moved to the MultiModuleController project folder 4.  More database cleanup work completed.
Parts:
- TURNOUT1, TURNOUT2: value PIN1 -> PIN0
Changed lines of the file:
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@@
 <element name="R4" library="SparkFun-Resistors" package="AXIAL-0.4" value="3.3K" x="53.34" y="13.97" rot="R180"/>
 <element name="R5" library="SparkFun-Resistors" package="AXIAL-0.4" value="3.3K" x="53.34" y="17.78" rot="R180"/>
-<element name="TURNOUT1" library="con-amp-quick" package="05P" value="PIN1" x="48.26" y="40.64" rot="R270">
+<element name="TURNOUT1" library="con-amp-quick" package="05P" value="PIN0" x="48.26" y="40.64" rot="R270">
 <attribute name="OC_FARNELL" value="unknown" x="48.26" y="40.64" size="1.778" layer="27" rot="R270" display="off"/>
 <attribute name="OC_NEWARK" value="unknown" x="48.26" y="40.64" size="1.778" layer="27" rot="R270" display="off"/>
@@
 <attribute name="MF" value="" x="48.26" y="40.64" size="1.778" layer="27" rot="R270" display="off"/>
 </element>
-<element name="TURNOUT2" library="con-amp-quick" package="05P" value="PIN1" x="22.86" y="40.64" rot="R270">
+<element name="TURNOUT2" library="con-amp-quick" package="05P" value="PIN0" x="22.86" y="40.64" rot="R270">
 <attribute name="OC_FARNELL" value="unknown" x="22.86" y="40.64" size="1.778" layer="27" rot="R270" display="off"/>
 <attribute name="OC_NEWARK" value="unknown" x="22.86" y="40.64" size="1.778" layer="27" rot="R270" display="off"/>
