File: eagle/ESP8266Controller/ESP8266Controller.sch (EAGLE design)
At the start: 18 parts, among them J1 POWER_JACKPTH

Commit message: 1.  More additions to the API 2.  Rename device.moduleIndex to device.port 3.  Begin work on new InputModule 4.  Module:  remove unused functions: 	virtual byte getDeviceCount(void) const = 0; 	virtual short getDeviceID(byte index) const = 0;
Parts:
- added EXTRA: PIN0, con-amp-quick:M04
- added POWER_LED1: 3.3, SparkFun-LED:LED5MM
- added R1: 220, SparkFun-Resistors:RESISTORPTH-1/4W
Connections:
- removed net N$34: U$1.GPIO14
- removed net N$35: U$1.GPIO12
- removed net N$36: U$1.GPIO2
- new net N$1: EXTRA.4, POWER_LED1.A, R1.2
- new net N$2: R1.1, U$1.GPIO12
- new net N$3: EXTRA.3, U$1.GPIO13
- net +3V3: now also EXTRA.2
- net GND: now also EXTRA.1, POWER_LED1.C
Changed lines of the file:
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@@
 <part name="I2C6" library="con-amp-quick" deviceset="M05" device="" value="PIN1"/>
 <part name="I2C7" library="con-amp-quick" deviceset="M05" device="" value="PIN1"/>
+<part name="GND2" library="SparkFun-Aesthetics" deviceset="GND" device=""/>
+<part name="+3V2" library="supply1" deviceset="+3V3" device=""/>
+<part name="R1" library="SparkFun-Resistors" deviceset="RESISTOR" device="PTH-1/4W" value="220"/>
+<part name="POWER_LED1" library="SparkFun-LED" deviceset="LED" device="5MM" value="3.3"/>
+<part name="EXTRA" library="con-amp-quick" deviceset="M04" device="" value="PIN0"/>
 </parts>
 <sheets>
@@
 <instance part="I2C6" gate="G$1" x="137.16" y="129.54" rot="R270"/>
 <instance part="I2C7" gate="G$1" x="137.16" y="139.7" rot="R270"/>
+<instance part="GND2" gate="1" x="20.32" y="76.2"/>
+<instance part="+3V2" gate="G$1" x="22.86" y="68.58" rot="R180"/>
+<instance part="R1" gate="G$1" x="2.54" y="53.34" rot="R90"/>
+<instance part="POWER_LED1" gate="G$1" x="2.54" y="73.66" rot="R180"/>
+<instance part="EXTRA" gate="G$1" x="22.86" y="91.44" rot="R270"/>
 </instances>
 <busses>
@@
 <wire x1="132.08" y1="121.92" x2="132.08" y2="132.08" width="0.1524" layer="91"/>
 <junction x="132.08" y="121.92"/>
+</segment>
+<segment>
+<pinref part="GND2" gate="1" pin="GND"/>
+<wire x1="20.32" y1="86.36" x2="20.32" y2="81.28" width="0.1524" layer="91"/>
+<pinref part="POWER_LED1" gate="G$1" pin="C"/>
+<wire x1="20.32" y1="81.28" x2="20.32" y2="78.74" width="0.1524" layer="91"/>
+<wire x1="2.54" y1="78.74" x2="2.54" y2="81.28" width="0.1524" layer="91"/>
+<wire x1="2.54" y1="81.28" x2="20.32" y2="81.28" width="0.1524" layer="91"/>
+<junction x="20.32" y="81.28"/>
+<pinref part="EXTRA" gate="G$1" pin="1"/>
 </segment>
 </net>
@@
 <junction x="134.62" y="121.92"/>
 </segment>
-</net>
-<net name="N$34" class="0">
-<segment>
-<pinref part="U$1" gate="G$1" pin="GPIO14"/>
-<wire x1="12.7" y1="45.72" x2="7.62" y2="45.72" width="0.1524" layer="91"/>
-</segment>
-</net>
-<net name="N$35" class="0">
-<segment>
-<pinref part="U$1" gate="G$1" pin="GPIO12"/>
-<wire x1="12.7" y1="43.18" x2="10.16" y2="43.18" width="0.1524" layer="91"/>
-</segment>
-</net>
-<net name="N$36" class="0">
-<segment>
-<pinref part="U$1" gate="G$1" pin="GPIO2"/>
-<wire x1="45.72" y1="43.18" x2="50.8" y2="43.18" width="0.1524" layer="91"/>
+<segment>
+<pinref part="+3V2" gate="G$1" pin="+3V3"/>
+<wire x1="22.86" y1="71.12" x2="22.86" y2="86.36" width="0.1524" layer="91"/>
+<pinref part="EXTRA" gate="G$1" pin="2"/>
 </segment>
 </net>
@@
 </segment>
 </net>
+<net name="N$2" class="0">
+<segment>
+<wire x1="2.54" y1="48.26" x2="2.54" y2="43.18" width="0.1524" layer="91"/>
+<pinref part="U$1" gate="G$1" pin="GPIO12"/>
+<wire x1="2.54" y1="43.18" x2="12.7" y2="43.18" width="0.1524" layer="91"/>
+<pinref part="R1" gate="G$1" pin="1"/>
+</segment>
+</net>
+<net name="N$3" class="0">
+<segment>
+<pinref part="U$1" gate="G$1" pin="GPIO13"/>
+<wire x1="12.7" y1="40.64" x2="5.08" y2="40.64" width="0.1524" layer="91"/>
+<wire x1="5.08" y1="40.64" x2="5.08" y2="63.5" width="0.1524" layer="91"/>
+<wire x1="5.08" y1="63.5" x2="25.4" y2="63.5" width="0.1524" layer="91"/>
+<wire x1="25.4" y1="86.36" x2="25.4" y2="63.5" width="0.1524" layer="91"/>
+<pinref part="EXTRA" gate="G$1" pin="3"/>
+</segment>
+</net>
+<net name="N$1" class="0">
+<segment>
+<pinref part="POWER_LED1" gate="G$1" pin="A"/>
+<pinref part="R1" gate="G$1" pin="2"/>
+<wire x1="2.54" y1="58.42" x2="2.54" y2="66.04" width="0.1524" layer="91"/>
+<wire x1="2.54" y1="66.04" x2="2.54" y2="71.12" width="0.1524" layer="91"/>
+<wire x1="2.54" y1="66.04" x2="27.94" y2="66.04" width="0.1524" layer="91"/>
+<wire x1="27.94" y1="66.04" x2="27.94" y2="86.36" width="0.1524" layer="91"/>
+<junction x="2.54" y="66.04"/>
+<pinref part="EXTRA" gate="G$1" pin="4"/>
+</segment>
+</net>

Commit message: 1.  Cleanup continues.  BlockController and the corresponding controller are deprecated along with SignalController and it's controller board.  These are replaced by the InputModule and OutputModule respectively 2.  TurnoutHandler moved to the MultiModuleController project folder 3.  Module moved to the MultiModuleController project folder 4.  More database cleanup work completed.
Parts:
- removed POWER_LED1: 3.3, SparkFun-LED:LED5MM
- EXTRA: value PIN0 -> (none)
- I2C, I2C1, I2C2, I2C3, I2C4, I2C5, I2C6, I2C7: value PIN1 -> (none)
Connections:
- net N$6 renamed SDA
- net N$8 renamed SCL
- net GND: no longer POWER_LED1.C
- net N$1: no longer POWER_LED1.A
- net N$2: now also U$1.GPIO2; no longer U$1.GPIO12
Other:
- note added: "I2C BUS"
Changed lines of the file:
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@@
 <part name="+3V7" library="supply1" deviceset="+3V3" device=""/>
 <part name="SUPPLY1" library="SparkFun-Aesthetics" deviceset="VCC" device=""/>
-<part name="I2C" library="con-amp-quick" deviceset="M05" device="" value="PIN1"/>
+<part name="I2C" library="con-amp-quick" deviceset="M05" device=""/>
 <part name="SUPPLY2" library="SparkFun-Aesthetics" deviceset="VCC" device=""/>
-<part name="I2C1" library="con-amp-quick" deviceset="M05" device="" value="PIN1"/>
-<part name="I2C2" library="con-amp-quick" deviceset="M05" device="" value="PIN1"/>
-<part name="I2C3" library="con-amp-quick" deviceset="M05" device="" value="PIN1"/>
-<part name="I2C4" library="con-amp-quick" deviceset="M05" device="" value="PIN1"/>
-<part name="I2C5" library="con-amp-quick" deviceset="M05" device="" value="PIN1"/>
-<part name="I2C6" library="con-amp-quick" deviceset="M05" device="" value="PIN1"/>
-<part name="I2C7" library="con-amp-quick" deviceset="M05" device="" value="PIN1"/>
+<part name="I2C1" library="con-amp-quick" deviceset="M05" device=""/>
+<part name="I2C2" library="con-amp-quick" deviceset="M05" device=""/>
+<part name="I2C3" library="con-amp-quick" deviceset="M05" device=""/>
+<part name="I2C4" library="con-amp-quick" deviceset="M05" device=""/>
+<part name="I2C5" library="con-amp-quick" deviceset="M05" device=""/>
+<part name="I2C6" library="con-amp-quick" deviceset="M05" device=""/>
+<part name="I2C7" library="con-amp-quick" deviceset="M05" device=""/>
 <part name="GND2" library="SparkFun-Aesthetics" deviceset="GND" device=""/>
 <part name="+3V2" library="supply1" deviceset="+3V3" device=""/>
 <part name="R1" library="SparkFun-Resistors" deviceset="RESISTOR" device="PTH-1/4W" value="220"/>
-<part name="POWER_LED1" library="SparkFun-LED" deviceset="LED" device="5MM" value="3.3"/>
-<part name="EXTRA" library="con-amp-quick" deviceset="M04" device="" value="PIN0"/>
+<part name="EXTRA" library="con-amp-quick" deviceset="M04" device=""/>
 </parts>
 <sheets>
 <sheet>
 <plain>
+<text x="73.66" y="53.34" size="1.778" layer="97">I2C BUS</text>
 </plain>
 <instances>
@@
 <instance part="I2C6" gate="G$1" x="137.16" y="129.54" rot="R270"/>
 <instance part="I2C7" gate="G$1" x="137.16" y="139.7" rot="R270"/>
-<instance part="GND2" gate="1" x="20.32" y="76.2"/>
-<instance part="+3V2" gate="G$1" x="22.86" y="68.58" rot="R180"/>
+<instance part="GND2" gate="1" x="17.78" y="78.74" rot="R270"/>
+<instance part="+3V2" gate="G$1" x="17.78" y="73.66" rot="R90"/>
 <instance part="R1" gate="G$1" x="2.54" y="53.34" rot="R90"/>
-<instance part="POWER_LED1" gate="G$1" x="2.54" y="73.66" rot="R180"/>
 <instance part="EXTRA" gate="G$1" x="22.86" y="91.44" rot="R270"/>
 </instances>
@@
 <segment>
 <pinref part="GND2" gate="1" pin="GND"/>
-<wire x1="20.32" y1="86.36" x2="20.32" y2="81.28" width="0.1524" layer="91"/>
-<pinref part="POWER_LED1" gate="G$1" pin="C"/>
-<wire x1="20.32" y1="81.28" x2="20.32" y2="78.74" width="0.1524" layer="91"/>
-<wire x1="2.54" y1="78.74" x2="2.54" y2="81.28" width="0.1524" layer="91"/>
-<wire x1="2.54" y1="81.28" x2="20.32" y2="81.28" width="0.1524" layer="91"/>
-<junction x="20.32" y="81.28"/>
+<wire x1="20.32" y1="86.36" x2="20.32" y2="78.74" width="0.1524" layer="91"/>
 <pinref part="EXTRA" gate="G$1" pin="1"/>
 </segment>
@@
 <segment>
 <pinref part="+3V2" gate="G$1" pin="+3V3"/>
-<wire x1="22.86" y1="71.12" x2="22.86" y2="86.36" width="0.1524" layer="91"/>
+<wire x1="20.32" y1="73.66" x2="22.86" y2="73.66" width="0.1524" layer="91"/>
+<wire x1="22.86" y1="73.66" x2="22.86" y2="86.36" width="0.1524" layer="91"/>
 <pinref part="EXTRA" gate="G$1" pin="2"/>
 </segment>
@@
 </segment>
 </net>
-<net name="N$6" class="0">
+<net name="SDA" class="0">
 <segment>
 <pinref part="R21" gate="G$1" pin="2"/>
@@
 <wire x1="142.24" y1="121.92" x2="142.24" y2="132.08" width="0.1524" layer="91"/>
 <junction x="142.24" y="121.92"/>
-</segment>
-</net>
-<net name="N$8" class="0">
+<label x="45.72" y="48.26" size="1.778" layer="95"/>
+</segment>
+</net>
+<net name="SCL" class="0">
 <segment>
 <pinref part="R20" gate="G$1" pin="2"/>
@@
 <wire x1="139.7" y1="121.92" x2="139.7" y2="132.08" width="0.1524" layer="91"/>
 <junction x="139.7" y="121.92"/>
+<label x="45.72" y="50.8" size="1.778" layer="95"/>
 </segment>
 </net>
 <net name="N$2" class="0">
 <segment>
-<wire x1="2.54" y1="48.26" x2="2.54" y2="43.18" width="0.1524" layer="91"/>
-<pinref part="U$1" gate="G$1" pin="GPIO12"/>
-<wire x1="2.54" y1="43.18" x2="12.7" y2="43.18" width="0.1524" layer="91"/>
 <pinref part="R1" gate="G$1" pin="1"/>
+<pinref part="U$1" gate="G$1" pin="GPIO2"/>
+<wire x1="45.72" y1="43.18" x2="50.8" y2="43.18" width="0.1524" layer="91"/>
+<wire x1="50.8" y1="43.18" x2="50.8" y2="27.94" width="0.1524" layer="91"/>
+<wire x1="50.8" y1="27.94" x2="2.54" y2="27.94" width="0.1524" layer="91"/>
+<wire x1="2.54" y1="27.94" x2="2.54" y2="48.26" width="0.1524" layer="91"/>
 </segment>
 </net>
@@
 <net name="N$1" class="0">
 <segment>
-<pinref part="POWER_LED1" gate="G$1" pin="A"/>
 <pinref part="R1" gate="G$1" pin="2"/>
 <wire x1="2.54" y1="58.42" x2="2.54" y2="66.04" width="0.1524" layer="91"/>
-<wire x1="2.54" y1="66.04" x2="2.54" y2="71.12" width="0.1524" layer="91"/>
 <wire x1="2.54" y1="66.04" x2="27.94" y2="66.04" width="0.1524" layer="91"/>
 <wire x1="27.94" y1="66.04" x2="27.94" y2="86.36" width="0.1524" layer="91"/>
-<junction x="2.54" y="66.04"/>
 <pinref part="EXTRA" gate="G$1" pin="4"/>
 </segment>

Commit message: 1.  Add jitter-detection to BlockDevice 2.  Add flashing pins to  ModuleData 3.  Move flashing pin code from PanelOutputDevice to OutputModule.  This insures pins blink at the same rate and same state. 4.  Fix flashing code for PanelInputDevice/OutputModule 5.  Remove unused code from PanelInputDevice 6.  fix jitter-detection code in TurnoutDevice 7.  New checkbox on StatusDialog allows enabling/disabling of server heartbeat messages 8.  Remove one of the I2C connections from the LCS Controller to make room for labels for the I2C pins 9.  Up build version to 19
Parts:
- removed I2C7: (no value), con-amp-quick:M05
Connections:
- net +3V3: no longer I2C7.2
- net GND: no longer I2C7.1
- net SCL: no longer I2C7.4
- net SDA: no longer I2C7.5
- net VCC: no longer I2C7.3
Changed lines of the file:
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@@
 <part name="I2C5" library="con-amp-quick" deviceset="M05" device=""/>
 <part name="I2C6" library="con-amp-quick" deviceset="M05" device=""/>
-<part name="I2C7" library="con-amp-quick" deviceset="M05" device=""/>
 <part name="GND2" library="SparkFun-Aesthetics" deviceset="GND" device=""/>
 <part name="+3V2" library="supply1" deviceset="+3V3" device=""/>
@@
 <instance part="I2C5" gate="G$1" x="137.16" y="116.84" rot="R270"/>
 <instance part="I2C6" gate="G$1" x="137.16" y="129.54" rot="R270"/>
-<instance part="I2C7" gate="G$1" x="137.16" y="139.7" rot="R270"/>
 <instance part="GND2" gate="1" x="17.78" y="78.74" rot="R270"/>
 <instance part="+3V2" gate="G$1" x="17.78" y="73.66" rot="R90"/>
@@
 <wire x1="132.08" y1="109.22" x2="132.08" y2="121.92" width="0.1524" layer="91"/>
 <junction x="132.08" y="109.22"/>
-<pinref part="I2C7" gate="G$1" pin="1"/>
 <wire x1="132.08" y1="121.92" x2="132.08" y2="132.08" width="0.1524" layer="91"/>
 <junction x="132.08" y="121.92"/>
@@
 <wire x1="134.62" y1="109.22" x2="134.62" y2="121.92" width="0.1524" layer="91"/>
 <junction x="134.62" y="109.22"/>
-<pinref part="I2C7" gate="G$1" pin="2"/>
 <wire x1="134.62" y1="121.92" x2="134.62" y2="132.08" width="0.1524" layer="91"/>
 <junction x="134.62" y="121.92"/>
@@
 <wire x1="137.16" y1="109.22" x2="137.16" y2="121.92" width="0.1524" layer="91"/>
 <junction x="137.16" y="109.22"/>
-<pinref part="I2C7" gate="G$1" pin="3"/>
 <wire x1="137.16" y1="121.92" x2="137.16" y2="132.08" width="0.1524" layer="91"/>
 <junction x="137.16" y="121.92"/>
@@
 <wire x1="142.24" y1="109.22" x2="142.24" y2="121.92" width="0.1524" layer="91"/>
 <junction x="142.24" y="109.22"/>
-<pinref part="I2C7" gate="G$1" pin="5"/>
 <wire x1="142.24" y1="121.92" x2="142.24" y2="132.08" width="0.1524" layer="91"/>
 <junction x="142.24" y="121.92"/>
@@
 <wire x1="139.7" y1="109.22" x2="139.7" y2="121.92" width="0.1524" layer="91"/>
 <junction x="139.7" y="109.22"/>
-<pinref part="I2C7" gate="G$1" pin="4"/>
 <wire x1="139.7" y1="121.92" x2="139.7" y2="132.08" width="0.1524" layer="91"/>
 <junction x="139.7" y="121.92"/>

Commit message: 1.  Add copyDevice to API 2.  Add modelChanged property to JSonModel
Parts:
- SERIAL: value PIN1 -> PIN0
Changed lines of the file:
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@@
 <part name="GND11" library="SparkFun-Aesthetics" deviceset="GND" device=""/>
 <part name="U$1" library="esp8266modules" deviceset="ESP12" device=""/>
-<part name="SERIAL" library="con-amp-quick" deviceset="M05" device="" value="PIN1"/>
+<part name="SERIAL" library="con-amp-quick" deviceset="M05" device="" value="PIN0"/>
 <part name="GND3" library="SparkFun-Aesthetics" deviceset="GND" device=""/>
 <part name="GND7" library="SparkFun-Aesthetics" deviceset="GND" device=""/>

Commit message: New Update!
1.  Documentation checked in
2.  Two new messages:  SYS_DEVICE_CONFIG_CHANGED and SYS_ROUTE_CONFIG_CHANGED are now sent out by the API whenever a route or a device's configuration is changed.  The controllers respond by downloading the updated route or the updated device configuration.  In the case of a device configuration change, the controller also downloads it's notification list just in case it has changed as well.
3.  TurnoutDetails.qml now has the DeviceProperties section displayed
4.  PanelOutputDevice now supports multiple routes.  When ONVALUE is set to 1, the LED remains ON if ANY of the routes are active.  When ONVALUE is set to 0, the LED is ON only if ALL routes are in-active.
Parts:
- added X1: 14867, con-4ucon:14867
Connections:
- net GND: now also X1.1
Changed lines of the file:
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@@
 <part name="R1" library="SparkFun-Resistors" deviceset="RESISTOR" device="PTH-1/4W" value="220"/>
 <part name="EXTRA" library="con-amp-quick" deviceset="M04" device=""/>
+<part name="X1" library="con-4ucon" deviceset="14867" device=""/>
 </parts>
 <sheets>
@@
 <instance part="R1" gate="G$1" x="2.54" y="53.34" rot="R90"/>
 <instance part="EXTRA" gate="G$1" x="22.86" y="91.44" rot="R270"/>
+<instance part="X1" gate="G$1" x="86.36" y="129.54" rot="R90"/>
 </instances>
 <busses>
@@
 <wire x1="132.08" y1="121.92" x2="132.08" y2="132.08" width="0.1524" layer="91"/>
 <junction x="132.08" y="121.92"/>
+<pinref part="X1" gate="G$1" pin="1"/>
+<wire x1="81.28" y1="127" x2="81.28" y2="121.92" width="0.1524" layer="91"/>
+<wire x1="81.28" y1="121.92" x2="132.08" y2="121.92" width="0.1524" layer="91"/>
 </segment>
 <segment>
